Commit message: 3D modelの各パーツの原点を調整

File: urdf/ic120.xacro (robot description, xacro)
@@ -3,6 +3,9 @@
   <xacro:property name="PI" value="3.1415926535" />
   <xacro:property name="temp_mass" value="100" />
-  <xacro:property name="model_offset_x" value="-1.5" />
-  <xacro:property name="model_offset_y" value="-3.1" />
+  <xacro:property name="base_mass" value="100" />
+  <xacro:property name="model_offset_x" value="3.1" />
+  <xacro:property name="model_offset_y" value="-1.5" />
+  <!-- <xacro:property name="model_offset_x" value="-1.5" />
+  <xacro:property name="model_offset_y" value="-3.1" /> -->
   <link name="base_link"/>
   <link name="track_frame_link">
@@ -11,5 +14,5 @@
         <mesh filename="package://ic120_model/mesh/track_frame.stl" />
       </geometry>
-      <origin rpy="0 0 0" xyz="${model_offset_x} ${model_offset_y} 0"/>
+      <origin rpy="0 0 ${PI/2}" xyz="${model_offset_x} ${model_offset_y} 0"/>
       <material name="Gray">
         <color rgba="0.7 0.7 0.7 1.0"/>
@@ -32,5 +35,5 @@
         <mesh filename="package://ic120_model/mesh/track_belt.stl" />
       </geometry>
-      <origin rpy="0 0 0" xyz="${model_offset_x} ${model_offset_y} 0"/>
+      <origin rpy="0 0 ${PI/2}" xyz="${model_offset_x} ${model_offset_y} 0"/>
       <material name="Black">
         <color rgba="0 0 0 1.0"/>
@@ -48,10 +51,10 @@
     <axis xyz="0 0 1" />
   </joint>
-  <link name="vessel_link">
+  <link name="upper_frame_link">
     <visual>
       <geometry>
-        <mesh filename="package://ic120_model/mesh/vessel.stl" />
+        <mesh filename="package://ic120_model/mesh/upper.stl" />
       </geometry>
-      <origin rpy="0 0 0" xyz="${model_offset_x} ${model_offset_y} 0"/>
+      <origin rpy="0 0 ${PI/2}" xyz="${model_offset_x} ${model_offset_y} 0"/>
       <material name="Teal">
         <color rgba="0 0.5 0.5 1.0"/>
@@ -63,8 +66,8 @@
     </inertial>
   </link>
-  <joint name="vessel_joint" type="fixed">
+  <joint name="upper_frame_joint" type="fixed">
     <origin xyz="0 0 0" rpy="0 0 0"/>
     <parent link="track_frame_link"/>
-    <child  link="vessel_link"/>
+    <child  link="upper_frame_link"/>
     <axis xyz="0 0 1" />
   </joint>
@@ -74,5 +77,5 @@
         <mesh filename="package://ic120_model/mesh/cabin.stl" />
       </geometry>
-      <origin rpy="0 0 0" xyz="${model_offset_x} ${model_offset_y} 0"/>
+      <origin rpy="0 0 ${PI/2}" xyz="${model_offset_x} ${model_offset_y} 0"/>
       <material name="Black">
         <color rgba="0 0 0 1.0"/>
@@ -95,5 +98,5 @@
         <mesh filename="package://ic120_model/mesh/cabin_window.stl" />
       </geometry>
-      <origin rpy="0 0 0" xyz="${model_offset_x} ${model_offset_y} 0"/>
+      <origin rpy="0 0 ${PI/2}" xyz="${model_offset_x} ${model_offset_y} 0"/>
       <material name="Gray">
         <color rgba="0.7 0.7 0.7 0.2"/>

Commit message: add vessel pin link for dump up

File: urdf/ic120.xacro (robot description, xacro)
@@ -114,3 +114,34 @@
     <axis xyz="0 0 1" />
   </joint>
+  <link name="vessel_pin_link">
+    <visual>
+      <geometry>
+        <box size="0.001 0.001 0.001" />
+      </geometry>
+      <origin rpy="0 0 0" xyz="0 0 0"/>
+      <material name="Gray">
+        <color rgba="0.7 0.7 0.7 0.2"/>
+      </material>
+    </visual>
+    <inertial>
+      <origin xyz="0 0 0" />
+      <mass value="1.0e-03" />
+      <inertia ixx="1.0e-03" ixy="0.0" ixz="0.0"
+               iyy="1.0e-03" iyz="0.0"
+               izz="1.0e-03" />
+    </inertial>
+  </link>
+  <joint name="vessel_pin_joint" type="revolute">
+    <origin xyz="-2 0 1.5" rpy="0 0 0"/>
+    <parent link="base_link"/>
+    <child  link="vessel_pin_link"/>
+    <axis xyz="0 1 0" />
+    <limit effort="1" lower="-3.14" upper="0" velocity="0.5"/>
+  </joint>
+  <link name="vessel_middle_link"/>
+  <joint name="vessel_middle_joint" type="fixed">
+    <origin xyz="1 0 1" rpy="0 0 0"/>
+    <parent link="vessel_pin_link"/>
+    <child  link="vessel_middle_link"/>
+  </joint>
 </robot>

Commit message: modify model weight and size

File: urdf/ic120.xacro (robot description, xacro)
@@ -2,6 +2,6 @@
 <robot name="ic120" xmlns:xacro="http://ros.org/wiki/xacro" >
   <xacro:property name="PI" value="3.1415926535" />
-  <xacro:property name="temp_mass" value="100" />
-  <xacro:property name="base_mass" value="100" />
+  <xacro:property name="temp_mass" value="1" />
+  <xacro:property name="base_mass" value="1" />
   <xacro:property name="model_offset_x" value="3.1" />
   <xacro:property name="model_offset_y" value="-1.5" />

File: urdf/ic120_gazebo.xacro (robot description, xacro)
@@ -38,5 +38,5 @@
       <collision>
         <geometry>
-          <cylinder radius="0.6" length="0.01" />
+          <cylinder radius="0.5" length="0.1" />
         </geometry>
       </collision>
@@ -51,22 +51,22 @@
   </xacro:macro>
   <!--Track(Multi Wheel) Definition-->
-  <xacro:wheel_macro prefix="left_middle_wheel"  parent="base_link" xyz="0 1 0.6"/>
-  <xacro:wheel_macro prefix="left_front1_wheel"  parent="base_link" xyz="0.5 1 0.6"/>
-  <xacro:wheel_macro prefix="left_front2_wheel"  parent="base_link" xyz="1 1 0.6"/>
-  <xacro:wheel_macro prefix="left_front3_wheel"  parent="base_link" xyz="1.5 1 0.6"/>
-  <xacro:wheel_macro prefix="left_rear1_wheel"  parent="base_link" xyz="-0.5 1 0.6"/>
-  <xacro:wheel_macro prefix="left_rear2_wheel"  parent="base_link" xyz="-1 1 0.6"/>
-  <xacro:wheel_macro prefix="left_rear3_wheel"  parent="base_link" xyz="-1.5 1 0.6"/>
-  <xacro:wheel_macro prefix="right_middle_wheel"  parent="base_link" xyz="0 -1 0.6"/>
-  <xacro:wheel_macro prefix="right_front1_wheel"  parent="base_link" xyz="0.5 -1 0.6"/>
-  <xacro:wheel_macro prefix="right_front2_wheel"  parent="base_link" xyz="1 -1 0.6"/>
-  <xacro:wheel_macro prefix="right_front3_wheel"  parent="base_link" xyz="1.5 -1 0.6"/>
-  <xacro:wheel_macro prefix="right_rear1_wheel"  parent="base_link" xyz="-0.5 -1 0.6"/>
-  <xacro:wheel_macro prefix="right_rear2_wheel"  parent="base_link" xyz="-1 -1 0.6"/>
-  <xacro:wheel_macro prefix="right_rear3_wheel"  parent="base_link" xyz="-1.5 -1 0.6"/>
+  <xacro:wheel_macro prefix="left_middle_wheel"  parent="base_link" xyz="0 1 0.5"/>
+  <xacro:wheel_macro prefix="left_front1_wheel"  parent="base_link" xyz="0.5 1 0.5"/>
+  <xacro:wheel_macro prefix="left_front2_wheel"  parent="base_link" xyz="1 1 0.5"/>
+  <xacro:wheel_macro prefix="left_front3_wheel"  parent="base_link" xyz="1.5 1 0.5"/>
+  <xacro:wheel_macro prefix="left_rear1_wheel"  parent="base_link" xyz="-0.5 1 0.5"/>
+  <xacro:wheel_macro prefix="left_rear2_wheel"  parent="base_link" xyz="-1 1 0.5"/>
+  <xacro:wheel_macro prefix="left_rear3_wheel"  parent="base_link" xyz="-1.5 1 0.5"/>
+  <xacro:wheel_macro prefix="right_middle_wheel"  parent="base_link" xyz="0 -1 0.5"/>
+  <xacro:wheel_macro prefix="right_front1_wheel"  parent="base_link" xyz="0.5 -1 0.5"/>
+  <xacro:wheel_macro prefix="right_front2_wheel"  parent="base_link" xyz="1 -1 0.5"/>
+  <xacro:wheel_macro prefix="right_front3_wheel"  parent="base_link" xyz="1.5 -1 0.5"/>
+  <xacro:wheel_macro prefix="right_rear1_wheel"  parent="base_link" xyz="-0.5 -1 0.5"/>
+  <xacro:wheel_macro prefix="right_rear2_wheel"  parent="base_link" xyz="-1 -1 0.5"/>
+  <xacro:wheel_macro prefix="right_rear3_wheel"  parent="base_link" xyz="-1.5 -1 0.5"/>
   <gazebo>
-    <plugin name="gazebo_ros_control" filename="libgazebo_ros_control.so">
-      <robotNamespace>/ic120</robotNamespace>
-    </plugin>
+    <plugin name="gazebo_ros_control" filename="libgazebo_ros_control.so"/>
+      <!-- <robotNamespace>/ic120</robotNamespace>
+    </plugin> -->
   </gazebo>
 </robot>

Commit message: separate 3d model into upper_frame and vessel

File: urdf/ic120.xacro (robot description, xacro)
@@ -54,5 +54,5 @@
     <visual>
       <geometry>
-        <mesh filename="package://ic120_model/mesh/upper.stl" />
+        <mesh filename="package://ic120_model/mesh/upper_frame.stl" />
       </geometry>
       <origin rpy="0 0 ${PI/2}" xyz="${model_offset_x} ${model_offset_y} 0"/>
@@ -117,9 +117,9 @@
     <visual>
       <geometry>
-        <box size="0.001 0.001 0.001" />
+        <mesh filename="package://ic120_model/mesh/vessel.stl" />
       </geometry>
-      <origin rpy="0 0 0" xyz="0 0 0"/>
-      <material name="Gray">
-        <color rgba="0.7 0.7 0.7 0.2"/>
+      <origin rpy="0 0 ${PI/2}" xyz="${model_offset_x+2.3} ${model_offset_y} -1.55"/>
+      <material name="Teal">
+        <color rgba="0 0.5 0.5 1.0"/>
       </material>
     </visual>
@@ -133,5 +133,5 @@
   </link>
   <joint name="vessel_pin_joint" type="revolute">
-    <origin xyz="-2 0 1.5" rpy="0 0 0"/>
+    <origin xyz="-2.30 0 1.55" rpy="0 0 0"/>
     <parent link="base_link"/>
     <child  link="vessel_pin_link"/>
@@ -139,9 +139,10 @@
     <limit effort="1" lower="-3.14" upper="0" velocity="0.5"/>
   </joint>
-  <link name="vessel_middle_link"/>
-  <joint name="vessel_middle_joint" type="fixed">
-    <origin xyz="1 0 1" rpy="0 0 0"/>
-    <parent link="vessel_pin_link"/>
-    <child  link="vessel_middle_link"/>
+  <link name="vessel_link"/>
+  <joint name="vessel_joint" type="fixed">
+  <origin xyz="-1.6 0 1.5" rpy="0 0 0"/>
+    <parent link="track_frame_link"/>
+    <child  link="vessel_link"/>
+    <axis xyz="0 0 1" />
   </joint>
 </robot>
