Commit message: change link name for vessel

File: ic120_description/urdf/ic120.xacro (robot description, xacro)
@@ -27,15 +27,15 @@
 	</link>
 	<!-- bucket axis -->
-	<joint name="container_pin_joint" type="revolute">
+	<joint name="vessel_pin_joint" type="revolute">
 		<origin xyz="-3.0153 0 0.94605"/>
 		<axis xyz="0 1 0"/>
 		<parent link="body_link"/>
-		<child link="container_pin_link"/>
+		<child link="vessel_pin_link"/>
 		<limit lower="${-radians(65)}" upper="0" effort="30" velocity="6.159937255"/>
 	</joint>
-	<link name="container_pin_link">
+	<link name="vessel_pin_link">
 		<visual>
 			<geometry>
-				<mesh filename="package://ic120_description/meshes/ic120-container.dae"/>
+				<mesh filename="package://ic120_description/meshes/ic120-vessel.dae"/>
 			</geometry>
 		</visual>
@@ -54,5 +54,5 @@
 		<parent link="body_link"/>
 		<child link="cylinder_head_link"/>
-		<mimic joint="container_pin_joint" multiplier="${radians(5.72)/radians(-65)}"/>
+		<mimic joint="vessel_pin_joint" multiplier="${radians(5.72)/radians(-65)}"/>
 	</joint>
 	<!-- cylinder outer angle -->
@@ -60,5 +60,5 @@
 		<plugin name="cylinder_head_joint_mimic_joint_plugin"
 				filename="libroboticsgroup_upatras_gazebo_mimic_joint_plugin.so">
-			<joint>container_pin_joint</joint>
+			<joint>vessel_pin_joint</joint>
 			<mimicJoint>cylinder_head_joint</mimicJoint>
 			<multiplier>${radians(5.72)/radians(-65)}</multiplier>
@@ -88,5 +88,5 @@
 		<axis xyz="-1.4989 0 0.51788"/>
 		<limit lower="-1" upper="1" effort="30" velocity="6.159937255"/>
-		<mimic joint="container_pin_joint" multiplier="${0.8/radians(-65)}"/>
+		<mimic joint="vessel_pin_joint" multiplier="${0.8/radians(-65)}"/>
 	</joint>
 	<!-- cylinder inner position -->
@@ -94,5 +94,5 @@
 		<plugin name="cylinder_joint_mimic_joint_plugin"
 				filename="libroboticsgroup_upatras_gazebo_mimic_joint_plugin.so">
-			<joint>container_pin_joint</joint>
+			<joint>vessel_pin_joint</joint>
 			<mimicJoint>cylinder_rod_prismatic_joint</mimicJoint>
 			<multiplier>${0.8/radians(-65)}</multiplier>
@@ -117,8 +117,8 @@
 	<transmission name="tran1">
 		<type>transmission_interface/SimpleTransmission</type>
-		<joint name="container_pin_joint">
+		<joint name="vessel_pin_joint">
 			<hardwareInterface>hardware_interface/EffortJointInterface</hardwareInterface>
 		</joint>
-		<actuator name="container_pin_joint_motor">
+		<actuator name="vessel_pin_joint_motor">
 			<hardwareInterface>hardware_interface/EffortJointInterface</hardwareInterface>
 			<mechanicalReduction>1</mechanicalReduction>

Commit message: add track's sprocket link and joint

File: ic120_description/urdf/ic120.xacro (robot description, xacro)
@@ -3,5 +3,5 @@
 	<xacro:property name="PI" value="3.1415926535" />
 	<!-- Import all Gazebo-customization elements, including Gazebo colors -->
-	<xacro:include filename="$(find ic120_description)/urdf/ic120.gazebo" />
+	<!-- <xacro:include filename="$(find ic120_description)/urdf/ic120.gazebo" /> -->
 	<!-- Import Rviz colors -->
 	<!-- <xacro:include filename="$(find ic120_description)/urdf/materials.xacro" /> -->
@@ -26,4 +26,20 @@
 		</inertial>
 	</link>
+	<!-- left sprocket axis -->
+	<joint name="sprocket_left_joint" type="continuous">
+		<origin xyz="-2.35 1 0.65"/>
+		<axis xyz="0 1 0"/>
+		<parent link="body_link"/>
+		<child link="left_sprocket_link"/>
+	</joint>
+	<link name="left_sprocket_link"/>
+	<!-- right sprocket axis -->
+	<joint name="sprocket_right_joint" type="continuous">
+		<origin xyz="-2.35 -1 0.65"/>
+		<axis xyz="0 1 0"/>
+		<parent link="body_link"/>
+		<child link="right_sprocket_link"/>
+	</joint>
+	<link name="right_sprocket_link"/>
 	<!-- bucket axis -->
 	<joint name="vessel_pin_joint" type="revolute">
